Commit message: folder reaarangement, new subproject on trajectory following

File: twolinkman_description/urdf/twolinkman.xacro (robot description, xacro)
@@ -211,5 +211,5 @@
   <joint
     name="load_joint"
-    type="fixed">
+    type="revolute">
     <origin
       xyz="0.02145 -0.29824 -0.0025016"
@@ -220,5 +220,10 @@
       link="load_link" />
     <axis
-      xyz="0 0 0" />
+      xyz="0 0 1" />
+		<limit
+		  effort="0"
+		  velocity="0"
+			lower="0"
+      upper="0"/>
   </joint>
 	<transmission name="rear_tran">
